File: hardware/kosmo-16-channel-sequencer-main-board/kosmo-16-channel-sequencer-main-board.kicad_sch (KiCad schematic)
At the start: 42 parts, among them J1 ROW1, J10 ROW10, J11 5V_IN, J12 STEP-SETTINGS, J13 MIDI-IN, J17 MIDI-OUT-2, J18 CLOCK-OUT, J19 RESET, J2 ROW2, J20 USB HOST, J21 CLOCK-IN, J3 ROW3, J30 EXTERNAL BUS, J31 MIDI-OUT-1, J4 ROW4, J5 ROW5, J6 ROW6, J7 ROW7, J8 ROW8, J9 ROW9, U11 6N138, U12 74HCT14, U2 Teensy4.1, U33 74AHCT125

Commit message: Split combined PCB into three one-board KiCad projects
The single kicad_pcb held all three boards in one netlist, which made
the shared power rails bleed across board outlines and produced one
panelised Gerber set instead of three per-board sets.

Now one project per board, each with a single outline:

  -main-board            83 x 295 mm   42 footprints  (Teensy, MIDI, 165s)
  -row-board            377 x  49 mm   57 footprints
  -steps-settings-board 385 x  95 mm   98 footprints

Each keeps its original root sheet as a thin wrapper around the one
sheet symbol, so hierarchical net paths (/row-board/..., /step-settings-board/...)
are unchanged and the PCB pad-net assignments stayed in sync.

Includes a per-board Gerber and drill export for each project.

Co-Authored-By: Claude Opus 5 <noreply@anthropic.com>
Other:
- removed sheet row-board
- removed sheet step-settings-board
