File: hardware/kosmo-16-channel-sequencer-main-board/kosmo-16-channel-sequencer-main-board.kicad_sch (KiCad schematic)
At the start: 42 parts, among them J1 ROW1, J10 ROW10, J11 5V_IN, J12 STEP-SETTINGS, J13 MIDI-IN, J17 MIDI-OUT-2, J18 CLOCK-OUT, J19 RESET, J2 ROW2, J20 USB HOST, J21 CLOCK-IN, J3 ROW3, J30 EXTERNAL BUS, J31 MIDI-OUT-1, J4 ROW4, J5 ROW5, J6 ROW6, J7 ROW7, J8 ROW8, J9 ROW9, U11 6N138, U12 74HCT14, U2 Teensy4.1, U33 74AHCT125

Commit message: house keeping
Parts:
- U33: footprint Package_DIP:DIP-12_W7.62mm -> Package_DIP:DIP-14_W7.62mm
Changed lines of the file:
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@@
 	)
 	(junction
+		(at 135.89 33.02)
+		(diameter 0)
+		(color 0 0 0 0)
+	)
+	(junction
 		(at 240.03 26.67)
 		(diameter 0)
@@
 	(wire
 		(pts
+			(xy 135.89 33.02) (xy 142.24 33.02)
+		)
+		(stroke
+			(width 0)
+			(type default)
+		)
+	)
+	(wire
+		(pts
 			(xy 349.25 189.23) (xy 365.76 189.23)
 		)
@@
 	(wire
 		(pts
-			(xy 130.81 33.02) (xy 142.24 33.02)
+			(xy 130.81 33.02) (xy 135.89 33.02)
 		)
 		(stroke
@@
 	)
 	(symbol
+		(lib_id "power:PWR_FLAG")
+		(at 135.89 33.02 0)
+		(unit 1)
+		(body_style 1)
+		(exclude_from_sim no)
+		(in_bom yes)
+		(on_board yes)
+		(in_pos_files yes)
+		(dnp no)
+		(fields_autoplaced yes)
+		(property "Reference" "#FLG07"
+			(at 135.89 31.115 0)
+			(hide yes)
+			(show_name no)
+			(do_not_autoplace no)
+			(effects
+				(font
+					(size 1.27 1.27)
+				)
+			)
+		)
+		(property "Value" "PWR_FLAG"
+			(at 135.89 27.94 0)
+			(show_name no)
+			(do_not_autoplace no)
+			(effects
+				(font
+					(size 1.27 1.27)
+				)
+			)
+		)
+		(property "Footprint" ""
+			(at 135.89 33.02 0)
+			(hide yes)
+			(show_name no)
+			(do_not_autoplace no)
+			(effects
+				(font
+					(size 1.27 1.27)
+				)
+			)
+		)
+		(property "Datasheet" ""
+			(at 135.89 33.02 0)
+			(hide yes)
+			(show_name no)
+			(do_not_autoplace no)
+			(effects
+				(font
+					(size 1.27 1.27)
+				)
+			)
+		)
+		(property "Description" "Special symbol for telling ERC where power comes from"
+			(at 135.89 33.02 0)
+			(hide yes)
+			(show_name no)
+			(do_not_autoplace no)
+			(effects
+				(font
+					(size 1.27 1.27)
+				)
+			)
+		)
+		(pin "1"
+		)
+		(instances
+			(project "kosmo-16-channel-sequencer-main-board"
+				(path "/a54f4241-b83c-42c9-8a43-a4038e61e150"
+					(reference "#FLG07")
+					(unit 1)
+				)
+			)
+		)
+	)
+	(symbol
 		(lib_id "Connector:Conn_01x04_Pin")
 		(at 274.32 127 0)
@@
 			)
 		)
-		(property "Footprint" "Package_DIP:DIP-12_W7.62mm"
+		(property "Footprint" "Package_DIP:DIP-14_W7.62mm"
 			(at 372.11 87.63 0)
 			(hide yes)
@@
 			)
 		)
-		(property "Footprint" "Package_DIP:DIP-12_W7.62mm"
+		(property "Footprint" "Package_DIP:DIP-14_W7.62mm"
 			(at 242.57 67.31 0)
 			(hide yes)
@@
 			)
 		)
-		(property "Footprint" "Package_DIP:DIP-12_W7.62mm"
+		(property "Footprint" "Package_DIP:DIP-14_W7.62mm"
 			(at 238.76 120.65 0)
 			(hide yes)
@@
 			)
 		)
-		(property "Footprint" "Package_DIP:DIP-12_W7.62mm"
+		(property "Footprint" "Package_DIP:DIP-14_W7.62mm"
 			(at 242.57 97.79 0)
 			(hide yes)
@@
 			)
 		)
-		(property "Footprint" "Package_DIP:DIP-12_W7.62mm"
+		(property "Footprint" "Package_DIP:DIP-14_W7.62mm"
 			(at 242.57 82.55 0)
 			(hide yes)
