File: hardware/kosmo-16-channel-sequencer-main-board/kosmo-16-channel-sequencer-main-board.kicad_pcb (KiCad board)
At the start: 2 copper layers, 83 x 295 mm, 42 parts, among them J1 ROW1, J10 ROW10, J11 5V_IN, J12 STEP-SETTINGS, J13 MIDI-IN, J17 MIDI-OUT-2, J18 CLOCK-OUT, J19 RESET, J2 ROW2, J20 USB HOST, J21 CLOCK-IN, J3 ROW3, J30 EXTERNAL BUS, J31 MIDI-OUT-1, J4 ROW4, J5 ROW5, J6 ROW6, J7 ROW7, J8 ROW8, J9 ROW9, U11 6N138, U12 74HCT14, U2 Teensy4.1, U33 74AHCT125

Commit message: added pcb labels
Other:
- board text added: "KOSMO 16 CHANNEL MIDI SEQUENCER"
- board text added: "MAIN BOARD REV 1.0"
Changed lines of the file:
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@@
+		)
+	)
+	(gr_text "MAIN BOARD REV 1.0"
+		(at 280 234.5 0)
+		(layer "F.SilkS")
+		(effects
+			(font
+				(size 1 1)
+				(thickness 0.1)
+			)
+			(justify left bottom)
+		)
+	)
+	(gr_text "KOSMO 16 CHANNEL MIDI SEQUENCER"
+		(at 280 233 0)
+		(layer "F.SilkS" knockout)
+		(effects
+			(font
+				(size 1 1)
+				(thickness 0.2)
+				(bold yes)
+			)
+			(justify left bottom)
 		)
 	)

Commit message: house keeping
Parts:
- U33: footprint Package_DIP:DIP-12_W7.62mm -> Package_DIP:DIP-14_W7.62mm
Routing:
- net /+5V: track 1158.6 -> 1193.6 mm
- net /MAX_CLK: track 341.6 -> 364.3 mm, vias 1 -> 3
- net Net-(U2-13_SCK_LED): track 60.9 -> 66.4 mm
- net Net-(U2-9_OUT1C): track 86.8 -> 91.9 mm
- net /MAX_LOAD_STEP_SETTINGS: track 182.1 -> 179.4 mm
- net GND: track 1174.4 -> 1173.9 mm, vias 1 -> 2

Commit message: fixed invalid net names
Changed lines of the file:
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@@
 			(effects
 				(font
-					(size 0.7 0.7)
+					(size 0.8 0.8)
 					(thickness 0.15)
 				)
@@
 			(effects
 				(font
-					(size 0.7 0.7)
+					(size 0.8 0.8)
 					(thickness 0.15)
 				)
