File: hardware/kosmo-16-channel-sequencer-row-board/kosmo-16-channel-sequencer-row-board.kicad_pcb (KiCad board)
At the start: 2 copper layers, 377 x 49 mm, 57 parts, among them J15 ROW-ANGLED, SW1 SW_Push, SW10 SW_Push, SW11 SW_Push, SW12 SW_Push, SW13 SW_Push, SW14 SW_Push, SW15 SW_Push, SW16 SW_Push, SW2 SW_Push, SW3 SW_Push, SW4 SW_Push, SW5 SW_Push, SW6 SW_Push, SW7 SW_Push, SW8 SW_Push, SW9 SW_Push, U1 MAX7219, U3 74HC165, U4 74HC165

Commit message: added pcb labels
Other:
- board text added: "CHANNEL BOARD REV 1.0"
- board text added: "KOSMO 16 CHANNEL MIDI SEQUENCER"

Commit message: fixed invalid net names
Connections:
- net /row-board/165_CLK renamed /165_CLK
- net /row-board/165_QH renamed /165_QH
- net /row-board/165_SER_IN renamed /165_SER_IN
- net /row-board/165_SH/LD renamed /165_SH/LD
- net /row-board/BTN_0 renamed /BTN_0
- net /row-board/BTN_1 renamed /BTN_1
- net /row-board/BTN_10 renamed /BTN_10
- net /row-board/BTN_11 renamed /BTN_11
- net /row-board/BTN_12 renamed /BTN_12
- net /row-board/BTN_13 renamed /BTN_13
- net /row-board/BTN_14 renamed /BTN_14
- net /row-board/BTN_15 renamed /BTN_15
- net /row-board/BTN_2 renamed /BTN_2
- net /row-board/BTN_3 renamed /BTN_3
- net /row-board/BTN_4 renamed /BTN_4
- net /row-board/BTN_5 renamed /BTN_5
- net /row-board/BTN_6 renamed /BTN_6
- net /row-board/BTN_7 renamed /BTN_7
- net /row-board/BTN_8 renamed /BTN_8
- net /row-board/BTN_9 renamed /BTN_9
- net /row-board/DIG_0 renamed /DIG_0
- net /row-board/DIG_1 renamed /DIG_1
- net /row-board/DIG_2 renamed /DIG_2
- net /row-board/DIG_3 renamed /DIG_3
- net /row-board/DIG_4 renamed /DIG_4
- net /row-board/DIG_5 renamed /DIG_5
- net /row-board/MAX_CLK renamed /MAX_CLK
- net /row-board/MAX_DIN renamed /MAX_DIN
- net /row-board/MAX_DOUT renamed /MAX_DOUT
- net /row-board/MAX_LOAD renamed /MAX_LOAD
- net /row-board/SEG_A renamed /SEG_A
- net /row-board/SEG_B renamed /SEG_B
- net /row-board/SEG_C renamed /SEG_C
- net /row-board/SEG_D renamed /SEG_D
- net /row-board/SEG_DP renamed /SEG_DP
- net /row-board/SEG_E renamed /SEG_E
- net /row-board/SEG_F renamed /SEG_F
- net /row-board/SEG_G renamed /SEG_G
