File: hardware/kosmo-16-channel-sequencer-steps-settings-board/kosmo-16-channel-sequencer-step-settings-board.kicad_pcb (KiCad board)
At the start: 2 copper layers, 384.6 x 94.6 mm, 98 parts, among them J14 STEP-SETTINGS-ANGLED, SW29 NOTE1, SW30 NOTE2, SW31 NOTE3, SW32 NOTE4, SW33 LENGTH, SW34 VOLUME, SW35 CC1, SW36 CC2, SW37 CC3, SW38 ENV, SW39 PC, SW40 TRIGGER, U10 74HC165, U28 MAX7219, U29 MAX7219, U30 MAX7219, U31 MAX7219, U32 MAX7219, U5 MAX7219, U6 74HC165, U7 74HC165, U8 74HC165, U9 74HC165

Commit message: added pcb labels
Other:
- board text added: "KOSMO 16 CHANNEL MIDI SEQUENCER"
- board text added: "STEP SETTINGS BOARD REV 1.0"
Changed lines of the file:
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@@
 		(tags "C Disc series Radial pin pitch 5.00mm diameter 5mm width 2.5mm Capacitor")
 		(property "Reference" "C15"
-			(at 2.5 -2.5 0)
+			(at 7.645861 1.038374 0)
 			(layer "F.SilkS")
 			(effects
@@
 		(tags "Resistor Axial_DIN0207 series Axial Horizontal pin pitch 7.62mm 0.25W = 1/4W length 6.3mm diameter 2.5mm")
 		(property "Reference" "R26"
-			(at 3.81 -2.37 0)
+			(at 0.854139 2.461626 0)
 			(layer "F.SilkS")
 			(effects
@@
 		(tags "Resistor Axial_DIN0207 series Axial Horizontal pin pitch 7.62mm 0.25W = 1/4W length 6.3mm diameter 2.5mm")
 		(property "Reference" "R42"
-			(at 3.81 -2.37 0)
+			(at -2.734139 0.038374 0)
 			(layer "F.SilkS")
 			(effects
@@
 		(tags "Resistor Axial_DIN0207 series Axial Horizontal pin pitch 7.62mm 0.25W = 1/4W length 6.3mm diameter 2.5mm")
 		(property "Reference" "R33"
-			(at 3.81 -2.37 0)
+			(at -3.044139 0.038374 0)
 			(layer "F.SilkS")
 			(effects
@@
 		(tags "CP Radial series Radial pin pitch 2.50mm diameter 6.3mm height 7mm Electrolytic Capacitor")
 		(property "Reference" "C14"
-			(at 1.25 -4.4 0)
+			(at 6.145861 -0.461626 0)
 			(layer "F.SilkS")
 			(effects
@@
 		(tags "SMD DIP DIL PDIP SMDIP 2.54mm 15.24mm 600mil")
 		(property "Reference" "U32"
-			(at 0 -16.3 0)
+			(at 11.734139 14.531626 0)
 			(layer "F.SilkS")
 			(effects
@@
 		(tags "Resistor Axial_DIN0207 series Axial Horizontal pin pitch 7.62mm 0.25W = 1/4W length 6.3mm diameter 2.5mm")
 		(property "Reference" "R60"
-			(at 3.81 -2.37 0)
+			(at -2.835861 0.961626 0)
 			(layer "F.SilkS")
 			(effects
@@
 		(tags "Resistor Axial_DIN0207 series Axial Horizontal pin pitch 7.62mm 0.25W = 1/4W length 6.3mm diameter 2.5mm")
 		(property "Reference" "R37"
-			(at 3.81 -2.37 0)
+			(at -2.55159 -0.171823 0)
 			(layer "F.SilkS")
 			(effects
@@
 		(tags "CP Radial series Radial pin pitch 2.50mm diameter 6.3mm height 7mm Electrolytic Capacitor")
 		(property "Reference" "C20"
-			(at 1.25 -4.4 90)
+			(at -0.038374 -4.354139 90)
 			(layer "F.SilkS")
 			(effects
@@
 		)
 	)
+	(gr_text "STEP SETTINGS BOARD REV 1.0"
+		(at 48 175 0)
+		(layer "F.SilkS")
+		(effects
+			(font
+				(size 1 1)
+				(thickness 0.1)
+			)
+			(justify left bottom)
+		)
+	)
+	(gr_text "KOSMO 16 CHANNEL MIDI SEQUENCER"
+		(at 47.5 173 0)
+		(layer "F.SilkS" knockout)
+		(effects
+			(font
+				(size 1 1)
+				(thickness 0.2)
+				(bold yes)
+			)
+			(justify left bottom)
+		)
+	)

Commit message: fixed invalid net names
Connections:
- net /step-settings-board/165_BTN_CLK renamed /165_BTN_CLK
- net /step-settings-board/165_BTN_QH renamed /165_BTN_QH
- net /step-settings-board/165_BTN_SH/LD renamed /165_BTN_SH/LD
- net /step-settings-board/165_ENC_CLK renamed /165_ENC_CLK
- net /step-settings-board/165_ENC_QH renamed /165_ENC_QH
- net /step-settings-board/165_ENC_SH/LD renamed /165_ENC_SH/LD
- net /step-settings-board/1_DIG_0 renamed /1_DIG_0
- net /step-settings-board/1_DIG_1 renamed /1_DIG_1
- net /step-settings-board/1_DIG_2 renamed /1_DIG_2
- net /step-settings-board/1_DIG_3 renamed /1_DIG_3
- net /step-settings-board/1_DIG_4 renamed /1_DIG_4
- net /step-settings-board/1_DIG_5 renamed /1_DIG_5
- net /step-settings-board/1_DIG_6 renamed /1_DIG_6
- net /step-settings-board/1_DIG_7 renamed /1_DIG_7
- net /step-settings-board/2_DIG_0 renamed /2_DIG_0
- net /step-settings-board/2_DIG_1 renamed /2_DIG_1
- net /step-settings-board/2_DIG_2 renamed /2_DIG_2
- net /step-settings-board/2_DIG_3 renamed /2_DIG_3
- net /step-settings-board/2_DIG_4 renamed /2_DIG_4
- net /step-settings-board/2_DIG_5 renamed /2_DIG_5
- net /step-settings-board/2_DIG_6 renamed /2_DIG_6
- net /step-settings-board/2_DIG_7 renamed /2_DIG_7
- net /step-settings-board/3_DIG_0 renamed /3_DIG_0
- net /step-settings-board/3_DIG_1 renamed /3_DIG_1
- net /step-settings-board/3_DIG_2 renamed /3_DIG_2
- net /step-settings-board/3_DIG_3 renamed /3_DIG_3
- net /step-settings-board/3_DIG_4 renamed /3_DIG_4
- net /step-settings-board/3_DIG_5 renamed /3_DIG_5
- net /step-settings-board/4_DIG_0 renamed /4_DIG_0
- net /step-settings-board/4_DIG_1 renamed /4_DIG_1
- net /step-settings-board/4_DIG_2 renamed /4_DIG_2
- net /step-settings-board/4_DIG_3 renamed /4_DIG_3
- net /step-settings-board/4_DIG_4 renamed /4_DIG_4
- net /step-settings-board/4_DIG_5 renamed /4_DIG_5
- net /step-settings-board/5_DIG_0 renamed /5_DIG_0
- net /step-settings-board/5_DIG_1 renamed /5_DIG_1
- net /step-settings-board/5_DIG_2 renamed /5_DIG_2
- net /step-settings-board/5_DIG_3 renamed /5_DIG_3
- net /step-settings-board/5_DIG_4 renamed /5_DIG_4
- net /step-settings-board/5_DIG_5 renamed /5_DIG_5
- net /step-settings-board/5_DIG_6 renamed /5_DIG_6
- net /step-settings-board/6_DIG_0 renamed /6_DIG_0
- net /step-settings-board/6_DIG_1 renamed /6_DIG_1
- net /step-settings-board/6_DIG_2 renamed /6_DIG_2
- net /step-settings-board/6_DIG_3 renamed /6_DIG_3
- net /step-settings-board/6_DIG_4 renamed /6_DIG_4
- net /step-settings-board/6_DIG_5 renamed /6_DIG_5
- net /step-settings-board/6_DIG_6 renamed /6_DIG_6
- net /step-settings-board/CC1_A renamed /CC1_A
- net /step-settings-board/CC1_B renamed /CC1_B
- net /step-settings-board/CC1_BTN renamed /CC1_BTN
- net /step-settings-board/CC2_A renamed /CC2_A
- net /step-settings-board/CC2_B renamed /CC2_B
- net /step-settings-board/CC2_BTN renamed /CC2_BTN
- net /step-settings-board/CC3_A renamed /CC3_A
- net /step-settings-board/CC3_B renamed /CC3_B
- net /step-settings-board/CC3_BTN renamed /CC3_BTN
- net /step-settings-board/ENV_A renamed /ENV_A
- net /step-settings-board/ENV_B renamed /ENV_B
- net /step-settings-board/ENV_BTN renamed /ENV_BTN
- net /step-settings-board/LENGTH_A renamed /LENGTH_A
- net /step-settings-board/LENGTH_B renamed /LENGTH_B
- net /step-settings-board/LENGTH_BTN renamed /LENGTH_BTN
- net /step-settings-board/MAX_CLK renamed /MAX_CLK
- net /step-settings-board/MAX_DIN renamed /MAX_DIN
- net /step-settings-board/MAX_DOUT renamed /MAX_DOUT
- net /step-settings-board/MAX_LOAD renamed /MAX_LOAD
- net /step-settings-board/NOTE1_A renamed /NOTE1_A
- net /step-settings-board/NOTE1_B renamed /NOTE1_B
- net /step-settings-board/NOTE1_BTN renamed /NOTE1_BTN
- net /step-settings-board/NOTE2_A renamed /NOTE2_A
- net /step-settings-board/NOTE2_B renamed /NOTE2_B
- net /step-settings-board/NOTE2_BTN renamed /NOTE2_BTN
- net /step-settings-board/NOTE3_A renamed /NOTE3_A
- net /step-settings-board/NOTE3_B renamed /NOTE3_B
- net /step-settings-board/NOTE3_BTN renamed /NOTE3_BTN
- net /step-settings-board/NOTE4_A renamed /NOTE4_A
- net /step-settings-board/NOTE4_B renamed /NOTE4_B
- net /step-settings-board/NOTE4_BTN renamed /NOTE4_BTN
- net /step-settings-board/PC_A renamed /PC_A
- net /step-settings-board/PC_B renamed /PC_B
- net /step-settings-board/PC_BTN renamed /PC_BTN
- net /step-settings-board/TRIGGER_A renamed /TRIGGER_A
- net /step-settings-board/TRIGGER_B renamed /TRIGGER_B
- net /step-settings-board/TRIGGER_BTN renamed /TRIGGER_BTN
- net /step-settings-board/VOLUME_A renamed /VOLUME_A
- net /step-settings-board/VOLUME_B renamed /VOLUME_B
- net /step-settings-board/VOLUME_BTN renamed /VOLUME_BTN
